Commit message: basic load management and controls

File: install/humanoid_control/share/humanoid_control/urdf/humanoid_32dof.urdf.xacro (robot description, xacro)
@@ -1,32 +1,70 @@
 <?xml version="1.0"?>
 <robot name="humanoid_32dof" xmlns:xacro="http://www.ros.org/wiki/xacro">
+  <!-- Materials -->
   <material name="silver"><color rgba="0.75 0.75 0.75 1.0"/></material>
   <material name="blue"><color rgba="0.0 0.5 0.8 1.0"/></material>
-  <link name="base_link"><visual><geometry><box size="0.2 0.3 0.2"/></geometry><material name="silver"/></visual></link>
-  <link name="torso"><visual><geometry><cylinder radius="0.12" length="0.4"/></geometry><origin xyz="0 0 0.2"/><material name="silver"/></visual></link>
-  <joint name="waist_yaw" type="revolute"><parent link="base_link"/><child link="torso"/><origin xyz="0 0 0.1"/><axis xyz="0 0 1"/><limit lower="-1.5" upper="1.5" effort="100" velocity="1.0"/></joint>
-  <link name="neck_link"><visual><geometry><cylinder radius="0.05" length="0.1"/></geometry><origin xyz="0 0 0.05"/><material name="silver"/></visual></link>
+  <material name="black"><color rgba="0.1 0.1 0.1 1.0"/></material>
+  <!-- VIRTUAL WORLD LINK (The Ground) -->
+  <link name="world"/>
+  <!-- VIRTUAL SLIDER JOINT (Allows Body to move Up/Down) -->
+  <joint name="virtual_root_z" type="prismatic">
+    <parent link="world"/>
+    <child link="base_link"/>
+    <origin xyz="0 0 0.95" rpy="0 0 0"/> <!-- Start 0.95m off ground -->
+    <axis xyz="0 0 1"/>
+    <limit lower="-1.0" upper="1.0" effort="1000" velocity="1.0"/>
+  </joint>
+  <!-- Base Link (Pelvis) -->
+  <link name="base_link">
+    <visual>
+      <geometry><box size="0.2 0.3 0.2"/></geometry>
+      <material name="silver"/>
+    </visual>
+  </link>
+  <!-- Torso -->
+  <link name="torso">
+    <visual>
+      <geometry><cylinder radius="0.12" length="0.4"/></geometry>
+      <origin xyz="0 0 0.2"/>
+      <material name="silver"/>
+    </visual>
+  </link>
+  <joint name="waist_yaw" type="revolute"><parent link="base_link"/><child link="torso"/><origin xyz="0 0 0.1"/><axis xyz="0 0 1"/><limit lower="-1.57" upper="1.57" effort="100" velocity="1.0"/></joint>
+  <!-- Neck -->
+  <link name="neck_link">
+    <visual>
+      <geometry><cylinder radius="0.05" length="0.1"/></geometry>
+      <origin xyz="0 0 0.05"/><material name="silver"/>
+    </visual>
+  </link>
   <joint name="neck_pitch" type="revolute"><parent link="torso"/><child link="neck_link"/><origin xyz="0 0 0.4"/><axis xyz="0 1 0"/><limit lower="-0.5" upper="0.5" effort="10" velocity="1.0"/></joint>
-  <link name="head"><visual><geometry><sphere radius="0.1"/></geometry><origin xyz="0 0 0.1"/><material name="silver"/></visual></link>
+  <link name="head">
+    <visual>
+      <geometry><sphere radius="0.1"/></geometry>
+      <origin xyz="0 0 0.1"/><material name="silver"/>
+    </visual>
+  </link>
   <joint name="neck_yaw" type="revolute"><parent link="neck_link"/><child link="head"/><origin xyz="0 0 0.1"/><axis xyz="0 0 1"/><limit lower="-1.0" upper="1.0" effort="10" velocity="1.0"/></joint>
+  <!-- Arms Macro -->
   <xacro:macro name="arm" params="side reflect">
     <link name="${side}_shoulder_link"><visual><geometry><sphere radius="0.08"/></geometry><material name="blue"/></visual></link>
-    <joint name="${side}_shoulder_roll" type="revolute"><parent link="torso"/><child link="${side}_shoulder_link"/><origin xyz="0 ${reflect * 0.18} 0.35"/><axis xyz="1 0 0"/><limit lower="-1.5" upper="1.5" effort="50" velocity="1.5"/></joint>
+    <joint name="${side}_shoulder_roll" type="revolute"><parent link="torso"/><child link="${side}_shoulder_link"/><origin xyz="0 ${reflect * 0.18} 0.35"/><axis xyz="1 0 0"/><limit lower="-1.57" upper="1.57" effort="50" velocity="1.5"/></joint>
     <link name="${side}_upper_arm"><visual><geometry><cylinder radius="0.06" length="0.3"/></geometry><origin xyz="0 0 -0.15"/><material name="silver"/></visual></link>
     <joint name="${side}_shoulder_pitch" type="revolute"><parent link="${side}_shoulder_link"/><child link="${side}_upper_arm"/><axis xyz="0 1 0"/><limit lower="-2.0" upper="2.0" effort="50" velocity="1.5"/></joint>
     <link name="${side}_forearm"><visual><geometry><cylinder radius="0.05" length="0.25"/></geometry><origin xyz="0 0 -0.125"/><material name="silver"/></visual></link>
     <joint name="${side}_elbow_pitch" type="revolute"><parent link="${side}_upper_arm"/><child link="${side}_forearm"/><origin xyz="0 0 -0.3"/><axis xyz="0 1 0"/><limit lower="-2.5" upper="0.0" effort="40" velocity="2.0"/></joint>
-    <link name="${side}_hand"><visual><geometry><box size="0.05 0.1 0.1"/></geometry><origin xyz="0 0 -0.05"/><material name="silver"/></visual></link>
-    <joint name="${side}_wrist_roll" type="revolute"><parent link="${side}_forearm"/><child link="${side}_hand"/><origin xyz="0 0 -0.25"/><axis xyz="1 0 0"/><limit lower="-1.5" upper="1.5" effort="10" velocity="2.0"/></joint>
+    <link name="${side}_hand"><visual><geometry><box size="0.05 0.1 0.1"/></geometry><origin xyz="0 0 -0.05"/><material name="black"/></visual></link>
+    <joint name="${side}_wrist_roll" type="revolute"><parent link="${side}_forearm"/><child link="${side}_hand"/><origin xyz="0 0 -0.25"/><axis xyz="1 0 0"/><limit lower="-1.57" upper="1.57" effort="10" velocity="2.0"/></joint>
   </xacro:macro>
   <xacro:arm side="left" reflect="1"/>
   <xacro:arm side="right" reflect="-1"/>
+  <!-- Legs Macro -->
   <xacro:macro name="leg" params="side reflect">
     <link name="${side}_thigh"><visual><geometry><cylinder radius="0.08" length="0.4"/></geometry><origin xyz="0 0 -0.2"/><material name="silver"/></visual></link>
-    <joint name="${side}_hip_pitch" type="revolute"><parent link="base_link"/><child link="${side}_thigh"/><origin xyz="0 ${reflect * 0.1} 0"/><axis xyz="0 1 0"/><limit lower="-1.0" upper="1.0" effort="100" velocity="1.0"/></joint>
+    <joint name="${side}_hip_pitch" type="revolute"><parent link="base_link"/><child link="${side}_thigh"/><origin xyz="0 ${reflect * 0.1} 0"/><axis xyz="0 1 0"/><limit lower="-1.5" upper="1.0" effort="100" velocity="1.0"/></joint>
     <link name="${side}_shin"><visual><geometry><cylinder radius="0.07" length="0.35"/></geometry><origin xyz="0 0 -0.175"/><material name="silver"/></visual></link>
-    <joint name="${side}_knee_pitch" type="revolute"><parent link="${side}_thigh"/><child link="${side}_shin"/><origin xyz="0 0 -0.4"/><axis xyz="0 1 0"/><limit lower="0.0" upper="2.0" effort="100" velocity="1.0"/></joint>
-    <link name="${side}_foot"><visual><geometry><box size="0.2 0.1 0.05"/></geometry><origin xyz="0.05 0 -0.025"/><material name="silver"/></visual></link>
-    <joint name="${side}_ankle_pitch" type="revolute"><parent link="${side}_shin"/><child link="${side}_foot"/><origin xyz="0 0 -0.35"/><axis xyz="0 1 0"/><limit lower="-0.5" upper="0.5" effort="50" velocity="1.0"/></joint>
+    <joint name="${side}_knee_pitch" type="revolute"><parent link="${side}_thigh"/><child link="${side}_shin"/><origin xyz="0 0 -0.4"/><axis xyz="0 1 0"/><limit lower="0.0" upper="2.5" effort="100" velocity="1.0"/></joint>
+    <link name="${side}_foot"><visual><geometry><box size="0.2 0.1 0.05"/></geometry><origin xyz="0.05 0 -0.025"/><material name="black"/></visual></link>
+    <joint name="${side}_ankle_pitch" type="revolute"><parent link="${side}_shin"/><child link="${side}_foot"/><origin xyz="0 0 -0.35"/><axis xyz="0 1 0"/><limit lower="-1.0" upper="1.0" effort="50" velocity="1.0"/></joint>
   </xacro:macro>
   <xacro:leg side="left" reflect="1"/>

Commit message: path planning added

File: install/humanoid_control/share/humanoid_control/urdf/humanoid_32dof.urdf.xacro (robot description, xacro)
@@ -1,50 +1,38 @@
 <?xml version="1.0"?>
 <robot name="humanoid_32dof" xmlns:xacro="http://www.ros.org/wiki/xacro">
-  <!-- Materials -->
   <material name="silver"><color rgba="0.75 0.75 0.75 1.0"/></material>
   <material name="blue"><color rgba="0.0 0.5 0.8 1.0"/></material>
   <material name="black"><color rgba="0.1 0.1 0.1 1.0"/></material>
-  <!-- VIRTUAL WORLD LINK (The Ground) -->
   <link name="world"/>
-  <!-- VIRTUAL SLIDER JOINT (Allows Body to move Up/Down) -->
+  <!-- VIRTUAL X (Forward/Back) -->
+  <link name="virtual_x_link"/>
+  <joint name="virtual_root_x" type="prismatic">
+    <parent link="world"/>
+    <child link="virtual_x_link"/>
+    <origin xyz="0 0 0" rpy="0 0 0"/>
+    <axis xyz="1 0 0"/> <limit lower="-5.0" upper="5.0" effort="1000" velocity="1.0"/>
+  </joint>
+  <!-- VIRTUAL Y (Left/Right) -->
+  <link name="virtual_y_link"/>
+  <joint name="virtual_root_y" type="prismatic">
+    <parent link="virtual_x_link"/>
+    <child link="virtual_y_link"/>
+    <origin xyz="0 0 0" rpy="0 0 0"/>
+    <axis xyz="0 1 0"/> <limit lower="-5.0" upper="5.0" effort="1000" velocity="1.0"/>
+  </joint>
+  <!-- VIRTUAL Z (Up/Down - Crouch) -->
   <joint name="virtual_root_z" type="prismatic">
-    <parent link="world"/>
+    <parent link="virtual_y_link"/>
     <child link="base_link"/>
-    <origin xyz="0 0 0.95" rpy="0 0 0"/> <!-- Start 0.95m off ground -->
-    <axis xyz="0 0 1"/>
-    <limit lower="-1.0" upper="1.0" effort="1000" velocity="1.0"/>
+    <origin xyz="0 0 0.95" rpy="0 0 0"/>
+    <axis xyz="0 0 1"/> <limit lower="-1.0" upper="1.0" effort="1000" velocity="1.0"/>
   </joint>
-  <!-- Base Link (Pelvis) -->
-  <link name="base_link">
-    <visual>
-      <geometry><box size="0.2 0.3 0.2"/></geometry>
-      <material name="silver"/>
-    </visual>
-  </link>
-  <!-- Torso -->
-  <link name="torso">
-    <visual>
-      <geometry><cylinder radius="0.12" length="0.4"/></geometry>
-      <origin xyz="0 0 0.2"/>
-      <material name="silver"/>
-    </visual>
-  </link>
+  <link name="base_link"><visual><geometry><box size="0.2 0.3 0.2"/></geometry><material name="silver"/></visual></link>
+  <link name="torso"><visual><geometry><cylinder radius="0.12" length="0.4"/></geometry><origin xyz="0 0 0.2"/><material name="silver"/></visual></link>
   <joint name="waist_yaw" type="revolute"><parent link="base_link"/><child link="torso"/><origin xyz="0 0 0.1"/><axis xyz="0 0 1"/><limit lower="-1.57" upper="1.57" effort="100" velocity="1.0"/></joint>
-  <!-- Neck -->
-  <link name="neck_link">
-    <visual>
-      <geometry><cylinder radius="0.05" length="0.1"/></geometry>
-      <origin xyz="0 0 0.05"/><material name="silver"/>
-    </visual>
-  </link>
+  <link name="neck_link"><visual><geometry><cylinder radius="0.05" length="0.1"/></geometry><origin xyz="0 0 0.05"/><material name="silver"/></visual></link>
   <joint name="neck_pitch" type="revolute"><parent link="torso"/><child link="neck_link"/><origin xyz="0 0 0.4"/><axis xyz="0 1 0"/><limit lower="-0.5" upper="0.5" effort="10" velocity="1.0"/></joint>
-  <link name="head">
-    <visual>
-      <geometry><sphere radius="0.1"/></geometry>
-      <origin xyz="0 0 0.1"/><material name="silver"/>
-    </visual>
-  </link>
+  <link name="head"><visual><geometry><sphere radius="0.1"/></geometry><origin xyz="0 0 0.1"/><material name="silver"/></visual></link>
   <joint name="neck_yaw" type="revolute"><parent link="neck_link"/><child link="head"/><origin xyz="0 0 0.1"/><axis xyz="0 0 1"/><limit lower="-1.0" upper="1.0" effort="10" velocity="1.0"/></joint>
-  <!-- Arms Macro -->
   <xacro:macro name="arm" params="side reflect">
     <link name="${side}_shoulder_link"><visual><geometry><sphere radius="0.08"/></geometry><material name="blue"/></visual></link>
@@ -59,5 +47,4 @@
   <xacro:arm side="left" reflect="1"/>
   <xacro:arm side="right" reflect="-1"/>
-  <!-- Legs Macro -->
   <xacro:macro name="leg" params="side reflect">
     <link name="${side}_thigh"><visual><geometry><cylinder radius="0.08" length="0.4"/></geometry><origin xyz="0 0 -0.2"/><material name="silver"/></visual></link>
